Commit message: feat: support Alicia impedance control

File: arx_d_can/models/Alicia_M_1_2_follower_ARX.urdf (robot description, URDF)
Before this commit: robot alicia_m_v1_2_follower_arx, 10 links, 9 joints
Joints:
- joint joint1: limit lower=-2.7475 upper=2.7475 effort=5 velocity=10 -> lower=-2.7475 upper=2.7475 effort=20 velocity=10
- joint joint2: limit lower=-3.14 upper=0 effort=5 velocity=10 -> lower=-3.14 upper=0 effort=20 velocity=10
- joint joint3: limit lower=-3.14 upper=0 effort=5 velocity=10 -> lower=-3.14 upper=0 effort=20 velocity=10
- joint joint4: limit lower=-1.8849555921538759 upper=1.562069680534925 effort=5 velocity=10 -> lower=-1.8849555921538759 upper=1.562069680534925 effort=10 velocity=10
- joint joint5: limit lower=-1.57 upper=1.57 effort=5 velocity=10 -> lower=-1.57 upper=1.57 effort=10 velocity=10
- joint joint6: limit lower=-2.791 upper=2.791 effort=5 velocity=10 -> lower=-2.791 upper=2.791 effort=10 velocity=10
