Commit message: Limit joint2 travel to 130 degrees

File: arx_d_can/models/yunyi_v1_0.urdf (robot description, URDF)
Before this commit: robot yunyi_v1_0, 21 links, 20 joints
Joints:
- joint l-joint2: limit lower=-0.174 upper=3.14 effort=20 velocity=10 -> lower=-0.174 upper=2.26892802759 effort=20 velocity=10
- joint r-joint2: limit lower=-3.14 upper=0.174 effort=20 velocity=10 -> lower=-2.26892802759 upper=0.174 effort=20 velocity=10

Commit message: Set joint6 limits to minus 45 and plus 60 degrees

File: arx_d_can/models/yunyi_v1_0.urdf (robot description, URDF)
Before this commit: robot yunyi_v1_0, 21 links, 20 joints
Joints:
- joint l-joint6: limit lower=-1.04 upper=1.04 effort=3 velocity=10 -> lower=-0.785398163397 upper=1.0471975512 effort=3 velocity=10
- joint r-joint6: limit lower=-1.04 upper=1.04 effort=3 velocity=10 -> lower=-0.785398163397 upper=1.0471975512 effort=3 velocity=10

Commit message: Reduce joint4 upper travel limit

File: arx_d_can/models/yunyi_v1_0.urdf (robot description, URDF)
Before this commit: robot yunyi_v1_0, 21 links, 20 joints
Joints:
- joint l-joint4: limit lower=-0.174 upper=1.918 effort=9 velocity=10 -> lower=-0.174 upper=1.81514242207 effort=9 velocity=10
- joint r-joint4: limit lower=-0.174 upper=1.918 effort=9 velocity=10 -> lower=-0.174 upper=1.81514242207 effort=9 velocity=10

Commit message: Enforce joint limits and verify motor disable

File: arx_d_can/models/yunyi_v1_0.urdf (robot description, URDF)
Before this commit: robot yunyi_v1_0, 21 links, 20 joints
Joints:
- joint l-joint4: limit lower=-0.174 upper=1.81514242207 effort=9 velocity=10 -> lower=-0.0872664625997 upper=1.57079632679 effort=9 velocity=10
- joint r-joint4: limit lower=-0.174 upper=1.81514242207 effort=9 velocity=10 -> lower=-0.0872664625997 upper=1.57079632679 effort=9 velocity=10

Commit message: Set Yunyi joint4 limits to 90 degrees

File: arx_d_can/models/yunyi_v1_0.urdf (robot description, URDF)
Before this commit: robot yunyi_v1_0, 21 links, 20 joints
Joints:
- joint l-joint4: limit lower=-0.0872664625997 upper=1.57079632679 effort=9 velocity=10 -> lower=-1.57079632679 upper=1.57079632679 effort=9 velocity=10
- joint r-joint4: limit lower=-0.0872664625997 upper=1.57079632679 effort=9 velocity=10 -> lower=-1.57079632679 upper=1.57079632679 effort=9 velocity=10

Commit message: Set Yunyi joint4 limits to minus 5 and 90 degrees

File: arx_d_can/models/yunyi_v1_0.urdf (robot description, URDF)
Before this commit: robot yunyi_v1_0, 21 links, 20 joints
Joints:
- joint l-joint4: limit lower=-1.57079632679 upper=1.57079632679 effort=9 velocity=10 -> lower=-0.0872664625997 upper=1.57079632679 effort=9 velocity=10
- joint r-joint4: limit lower=-1.57079632679 upper=1.57079632679 effort=9 velocity=10 -> lower=-0.0872664625997 upper=1.57079632679 effort=9 velocity=10

Commit message: Set Yunyi joint3 limits to plus-minus 145 degrees

File: arx_d_can/models/yunyi_v1_0.urdf (robot description, URDF)
Before this commit: robot yunyi_v1_0, 21 links, 20 joints
Joints:
- joint l-joint3: limit lower=-1.57 upper=1.57 effort=9 velocity=10 -> lower=-2.53072741539 upper=2.53072741539 effort=9 velocity=10
- joint r-joint3: limit lower=-1.57 upper=1.57 effort=9 velocity=10 -> lower=-2.53072741539 upper=2.53072741539 effort=9 velocity=10

Commit message: feat: simplify Yunyi SDK and adopt native safety runtime

File: arx_d_can/models/yunyi_v1_0.urdf (robot description, URDF)
Before this commit: robot yunyi_v1_0, 21 links, 20 joints
Links:
- link base_link: mass 0.71247791262477 -> 0.694702957982967
- link l-base-link: mass 0.68389726503575 -> 0
- link l-link1: mass 0.602091921859626 -> 0.612628872562558
- link l-link2: mass 0.585710853592396 -> 0.791808015126076
- link l-link3: mass 0.788681077794546 -> 0.842434356423893
- link l-link4: mass 0.114096528744517 -> 0.117703346646349
- link l-link5: mass 0.818152596294269 -> 0.818152596601028
- link l-link6: mass 0.32096469253304 -> 0.320964692532981
- link l-link7: mass 0.467084017740121 -> 0.467084017740573
- link l-link8: mass 0.0243852131463264 -> 0.0290810458194532
- link l-link9: mass 0.0243852131463263 -> 0.0290810458548977
- link r-base-link: mass 0.523482694754592 -> 0.521980069832523
- link r-link1: mass 0.470540450754261 -> 0.48001
- link r-link2: mass 0.585710853592397 -> 0.58736
- link r-link3: mass 0.576568672234304 -> 0.611557224869322
- link r-link4: mass 0.114096514178463 -> 0.195867906346611
- link r-link5: mass 0.699252924274787 -> 0.699252923462321
- link r-link6: mass 0.320964706156219 -> 0.320964693534996
- link r-link7: mass 0.467084018342305 -> 0.176907351254231
- link r-link8: mass 0.0243852090898284 -> 0.0290810458933222
- link r-link9: mass 0.0243851843627102 -> 0.0290810458523318
Joints:
- joint l-base-joint: axis 0 0 0 -> (none); origin xyz=0 0.055 0.615 rpy=0 0 0 -> xyz=0 0.0475 0.615 rpy=0 0 0
- joint l-joint1: limit lower=-2.7475 upper=2.7475 effort=20 velocity=10 -> lower=-2.745 upper=2.745 effort=40 velocity=16; origin xyz=5e-05 0.1241 0.017933 rpy=0.260207346415 -4.64237005026e-07 3.548052552e-06 -> xyz=4.99999999996615E-05 0.119492997382172 0.0187095589940774 rpy=0.261799387799152 0 0
- joint l-joint2: axis 0.999999999996 2.72232798693e-06 -1.29497898547e-07 -> 1 0 0; limit lower=-0.174 upper=2.26892802759 effort=20 velocity=10 -> lower=-0.3489 upper=2.2678 effort=40 velocity=16; origin xyz=0.030291 0.061 -1.47354549439e-08 rpy=-0.260207346415 -4.64237005026e-07 -3.548052552e-06 -> xyz=-5.0000000000329E-05 0.0579999999999999 0 rpy=-0.261799387799152 0 0
- joint l-joint3: axis -1.20835140189e-07 -0.0031779554119 -0.999994950287 -> 0 0 -1; limit lower=-2.53072741539 upper=2.53072741539 effort=9 velocity=10 -> lower=-2.5294 upper=2.5294 effort=27 velocity=5; origin xyz=-0.0270000149267 -0.000189559333477 -0.119249845959 rpy=0 0 0 -> xyz=0.00434139983447429 0.00799999999863457 -0.11925 rpy=0 0 0
- joint l-joint4: axis 2.72271149599e-06 -0.999994950283 0.00317795541156 -> 0 -1 0; limit lower=-0.0872664625997 upper=1.57079632679 effort=9 velocity=10 -> lower=-0.1744 upper=2.2678 effort=27 velocity=5; origin xyz=1.14910866617e-08 0 -0.13409188129 rpy=0 0 0 -> xyz=0.00719572519347152 0.000125000001366032 -0.134000000000001 rpy=0 0 0
- joint l-joint5: axis 3.55666303496e-06 -0.00476324991493 -0.999988655654 -> 0 0 1; limit lower=-2.09 upper=2.09 effort=3 velocity=10 -> lower=-2.0933 upper=2.0933 effort=7 velocity=20; origin xyz=2.66405097865e-07 0 -0.0519043987523 rpy=0 0 0 -> xyz=-0.00983268534763712 0.000750000000000084 -0.059 rpy=0 0 0
- joint l-joint6: axis 6.3903025017e-06 -0.999988690606 0.0047559036059 -> 0 -1 0; limit lower=-0.785398163397 upper=1.0471975512 effort=3 velocity=10 -> lower=-0.785 upper=0.785 effort=7 velocity=20; origin xyz=5.51282770418e-07 -0.00220439902431 -0.154998241626 rpy=0 0 0 -> xyz=0 0 -0.155 rpy=0 0 0
- joint l-joint7: axis 0.99999999999 2.73397159405e-06 3.54365386726e-06 -> 1 0 0; limit lower=-1.04 upper=1.04 effort=3 velocity=10 -> lower=-1.3956 upper=1.3956 effort=7 velocity=20
- joint l-joint8: axis 6.39030535904e-06 -0.999988708069 0.00475223044231 -> 0 -1 0; origin xyz=-0.00399922970935 -0.0513459906502 -0.177757827974 rpy=0 0 0 -> xyz=-0.00399999999999219 -0.0504999999999951 -0.178 rpy=0 0 0
- joint l-joint9: axis -9.56104640758e-07 -0.999988708089 0.00475223041627 -> 0 -1 0; origin xyz=-0.00399950413517 0.0496528671028 -0.178238174236 rpy=0 0 0 -> xyz=-0.0039999999999937 0.050500000000005 -0.178 rpy=0 0 0
- joint r-base-joint: axis 0 0 0 -> (none); origin xyz=0 -0.055 0.615 rpy=0 0 0 -> xyz=0 -0.0475 0.615 rpy=0 0 0
- joint r-joint1: axis 0 1 0 -> 0 -1 0; limit lower=-2.7475 upper=2.7475 effort=20 velocity=10 -> lower=-2.745 upper=2.745 effort=40 velocity=16; origin xyz=5e-05 -0.1241 0.017933 rpy=-0.26338530718 4.69973431244e-07 3.54805953611e-06 -> xyz=5E-05 -0.11949 0.01871 rpy=-0.261799387799152 0 0
- joint r-joint2: axis 0.999999999989 4.62369474003e-06 -1.32519135564e-07 -> 1 0 0; limit lower=-2.26892802759 upper=0.174 effort=20 velocity=10 -> lower=-2.2678 upper=0.3489 effort=40 velocity=16; origin xyz=0.0292189990116 -0.061 0.00205611404559 rpy=0.26338530718 4.69973431244e-07 -3.54805953611e-06 -> xyz=-5E-05 -0.058 0 rpy=0.261799387799152 0 0
- joint r-joint3: axis 3.54803288537e-06 -0.00158897969971 -0.999998737565 -> 0 0 -1; limit lower=-2.53072741539 upper=2.53072741539 effort=9 velocity=10 -> lower=-2.5294 upper=2.5294 effort=27 velocity=5; origin xyz=-0.0259280127149 -0.000724927112191 -0.121238997916 rpy=0 0 0 -> xyz=0.0043414 -0.008 -0.11925 rpy=0 0 0
- joint r-joint4: axis 1.16496372423e-06 -0.99999874339 0.00158531275793 -> 0 1 0; limit lower=-0.0872664625997 upper=1.57079632679 effort=9 velocity=10 -> lower=-0.1744 upper=2.2678 effort=27 velocity=5; origin xyz=6.10994344404e-07 0 -0.134203551484 rpy=0 0 0 -> xyz=0.0071957 0 -0.134 rpy=0 0 0
- joint r-joint5: axis 0.0583344128702 -0.00158254516859 -0.998295843839 -> 0 0 1; limit lower=-2.09 upper=2.09 effort=3 velocity=10 -> lower=-2.0933 upper=2.0933 effort=7 velocity=20; origin xyz=0.00303335452008 0 -0.0519589432624 rpy=0 0 0 -> xyz=-0.00983268534763703 -0.000874999999999626 -0.059 rpy=0 0 0
- joint r-joint6: axis 1.16496372423e-06 -0.99999874339 0.00158531275793 -> 0 -1 0; limit lower=-0.785398163397 upper=1.0471975512 effort=3 velocity=10 -> lower=-0.785 upper=0.785 effort=7 velocity=20; origin xyz=0.00904183399488 0.000334091695669 -0.154735855795 rpy=0 0 0 -> xyz=0 0 -0.155 rpy=0 0 0
- joint r-joint7: axis -0.998297099839 -9.73144305398e-05 -0.0583343036577 -> 1 0 0; limit lower=-1.04 upper=1.04 effort=3 velocity=10 -> lower=-1.3956 upper=1.3956 effort=7 velocity=20
- joint r-joint8: axis 8.49885691213e-06 -0.999998736844 0.0015894145074 -> 0 -1 0; origin xyz=0.00639067531362 -0.0507820184343 -0.177849684612 rpy=0 0 0 -> xyz=-0.004 -0.0505 -0.178 rpy=0 0 0
- joint r-joint9: axis 1.16495712717e-06 -0.99999873756 0.00158898595948 -> 0 -1 0; origin xyz=0.0063901872896 0.0502178546126 -0.178009822843 rpy=0 0 0 -> xyz=-0.004 0.0505 -0.178 rpy=0 0 0

Commit message: feat: adopt deterministic runtime shutdown

File: arx_d_can/models/yunyi_v1_0.urdf (robot description, URDF)
Before this commit: robot yunyi_v1_0, 21 links, 20 joints
Joints:
- joint r-joint4: axis 0 1 0 -> 0 -1 0

Commit message: Upgrade SDK to Runtime ABI 3.0

File: arx_d_can/models/yunyi_v1_0.urdf (robot description, URDF)
Before this commit: robot yunyi_v1_0, 21 links, 20 joints
Links:
- added link l-tool0
- added link r-tool0
Joints:
- added joint l-tool0-fixed-joint: type fixed, parent l-link7, child l-tool0, origin xyz=-0.004 0 -0.178 rpy=0 0 0
- added joint r-tool0-fixed-joint: type fixed, parent r-link7, child r-tool0, origin xyz=-0.004 0 -0.178 rpy=0 0 0

Commit message: release: prepare Articore SDK 0.3.2

File: arx_d_can/models/yunyi_v1_0.urdf (robot description, URDF)
Before this commit: robot yunyi_v1_0, 23 links, 22 joints
Joints:
- joint r-joint1: axis 0 -1 0 -> 0 1 0
